File: f3_backplane.kicad_sch (KiCad schematic)
At the start: 4 parts

Commit message: More routing
Parts:
- H1, H2, H3, H4: footprint MountingHole:MountingHole_3.5mm_Pad_Via -> Mounting:MountingHole_3.5mm_Pad_Via_With_Alignment_Hole
Other:
- added sheet SATA1 (sata.kicad_sch)
- added sheet SATA2 (sata.kicad_sch)
Changed lines of the file:
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@@
+    (stroke (width 0) (type default))
+  )
+  (wire (pts (xy 64.77 85.09) (xy 88.9 85.09))
+    (stroke (width 0) (type default))
+  )
+  (wire (pts (xy 64.77 67.31) (xy 88.9 67.31))
+    (stroke (width 0) (type default))
+  )
+  (wire (pts (xy 64.77 92.71) (xy 88.9 92.71))
     (stroke (width 0) (type default))
   )
@@
     (stroke (width 0) (type default))
   )
+  (wire (pts (xy 64.77 74.93) (xy 88.9 74.93))
+    (stroke (width 0) (type default))
+  )
   (wire (pts (xy 64.77 118.11) (xy 88.9 118.11))
     (stroke (width 0) (type default))
@@
     (stroke (width 0) (type default))
   )
+  (wire (pts (xy 64.77 90.17) (xy 88.9 90.17))
+    (stroke (width 0) (type default))
+  )
   (wire (pts (xy 64.77 110.49) (xy 88.9 110.49))
     (stroke (width 0) (type default))
@@
     (stroke (width 0) (type default))
   )
+  (wire (pts (xy 64.77 69.85) (xy 88.9 69.85))
+    (stroke (width 0) (type default))
+  )
   (wire (pts (xy 25.4 177.8) (xy 25.4 179.07))
     (stroke (width 0) (type default))
@@
     (stroke (width 0) (type default))
   )
+  (wire (pts (xy 64.77 72.39) (xy 88.9 72.39))
+    (stroke (width 0) (type default))
+  )
   (wire (pts (xy 63.5 177.8) (xy 63.5 179.07))
     (stroke (width 0) (type default))
@@
     (stroke (width 0) (type default))
   )
+  (wire (pts (xy 64.77 87.63) (xy 88.9 87.63))
+    (stroke (width 0) (type default))
+  )
   (wire (pts (xy 64.77 113.03) (xy 88.9 113.03))
     (stroke (width 0) (type default))
@@
     (effects (font (size 1.27 1.27)) (justify left bottom))
   )
+  (label "SATA1_A+" (at 66.04 67.31 0) (fields_autoplaced)
+    (effects (font (size 1.27 1.27)) (justify left bottom))
+  )
+  (label "SATA2_A+" (at 66.04 85.09 0) (fields_autoplaced)
+    (effects (font (size 1.27 1.27)) (justify left bottom))
+  )
   (label "PCIE_TX+" (at 66.04 102.87 0) (fields_autoplaced)
     (effects (font (size 1.27 1.27)) (justify left bottom))
@@
     (effects (font (size 1.27 1.27)) (justify left bottom))
   )
+  (label "SATA2_B-" (at 66.04 92.71 0) (fields_autoplaced)
+    (effects (font (size 1.27 1.27)) (justify left bottom))
+  )
+  (label "SATA1_A-" (at 66.04 69.85 0) (fields_autoplaced)
+    (effects (font (size 1.27 1.27)) (justify left bottom))
+  )
   (label "PCIE_REFCLK-" (at 66.04 115.57 0) (fields_autoplaced)
     (effects (font (size 1.27 1.27)) (justify left bottom))
   )
+  (label "SATA2_A-" (at 66.04 87.63 0) (fields_autoplaced)
+    (effects (font (size 1.27 1.27)) (justify left bottom))
+  )
   (label "PERST#" (at 66.04 118.11 0) (fields_autoplaced)
     (effects (font (size 1.27 1.27)) (justify left bottom))
   )
+  (label "SATA1_B-" (at 66.04 74.93 0) (fields_autoplaced)
+    (effects (font (size 1.27 1.27)) (justify left bottom))
+  )
+  (label "SATA1_B+" (at 66.04 72.39 0) (fields_autoplaced)
+    (effects (font (size 1.27 1.27)) (justify left bottom))
+  )
+  (label "SATA2_B+" (at 66.04 90.17 0) (fields_autoplaced)
+    (effects (font (size 1.27 1.27)) (justify left bottom))
+  )
   (symbol (lib_id "Mechanical:MountingHole_Pad") (at 38.1 175.26 0) (unit 1)
     (in_bom yes) (on_board yes) (dnp no) (fields_autoplaced)
@@
       (effects (font (size 1.27 1.27)) (justify left))
     )
-    (property "Footprint" "MountingHole:MountingHole_3.5mm_Pad_Via" (at 38.1 175.26 0)
+    (property "Footprint" "Mounting:MountingHole_3.5mm_Pad_Via_With_Alignment_Hole" (at 38.1 175.26 0)
       (effects (font (size 1.27 1.27)) hide)
     )
@@
       (effects (font (size 1.27 1.27)) (justify left))
     )
-    (property "Footprint" "MountingHole:MountingHole_3.5mm_Pad_Via" (at 50.8 175.26 0)
+    (property "Footprint" "Mounting:MountingHole_3.5mm_Pad_Via_With_Alignment_Hole" (at 50.8 175.26 0)
       (effects (font (size 1.27 1.27)) hide)
     )
@@
       (effects (font (size 1.27 1.27)) (justify left))
     )
-    (property "Footprint" "MountingHole:MountingHole_3.5mm_Pad_Via" (at 25.4 175.26 0)
+    (property "Footprint" "Mounting:MountingHole_3.5mm_Pad_Via_With_Alignment_Hole" (at 25.4 175.26 0)
       (effects (font (size 1.27 1.27)) hide)
     )
@@
       (effects (font (size 1.27 1.27)) (justify left))
     )
-    (property "Footprint" "MountingHole:MountingHole_3.5mm_Pad_Via" (at 63.5 175.26 0)
+    (property "Footprint" "Mounting:MountingHole_3.5mm_Pad_Via_With_Alignment_Hole" (at 63.5 175.26 0)
       (effects (font (size 1.27 1.27)) hide)
     )
@@
       )
     )
+  )
+  (sheet (at 88.9 82.55) (size 19.05 12.7) (fields_autoplaced)
+    (stroke (width 0.1524) (type solid))
+    (fill (color 0 0 0 0.0000))
+    (property "Sheetname" "SATA2" (at 88.9 81.8384 0)
+      (effects (font (size 1.27 1.27)) (justify left bottom))
+    )
+    (property "Sheetfile" "sata.kicad_sch" (at 88.9 95.8346 0)
+      (effects (font (size 1.27 1.27)) (justify left top))
+    )
+    (pin "SATA_A+" input (at 88.9 85.09 180)
+      (effects (font (size 1.27 1.27)) (justify left))
+    )
+    (pin "SATA_A-" input (at 88.9 87.63 180)
+      (effects (font (size 1.27 1.27)) (justify left))
+    )
+    (pin "SATA_B+" input (at 88.9 90.17 180)
+      (effects (font (size 1.27 1.27)) (justify left))
+    )
+    (pin "SATA_B-" input (at 88.9 92.71 180)
+      (effects (font (size 1.27 1.27)) (justify left))
+    )
+    (instances
+      (project "f3_backplane"
+        (path "/a299def6-d097-4d1a-85e0-73dfb51409a1" (page "5"))
+      )
+    )
+  )
+  (sheet (at 88.9 64.77) (size 19.05 12.7) (fields_autoplaced)
+    (stroke (width 0.1524) (type solid))
+    (fill (color 0 0 0 0.0000))
+    (property "Sheetname" "SATA1" (at 88.9 64.0584 0)
+      (effects (font (size 1.27 1.27)) (justify left bottom))
+    )
+    (property "Sheetfile" "sata.kicad_sch" (at 88.9 78.0546 0)
+      (effects (font (size 1.27 1.27)) (justify left top))
+    )
+    (pin "SATA_A+" input (at 88.9 67.31 180)
+      (effects (font (size 1.27 1.27)) (justify left))
+    )
+    (pin "SATA_A-" input (at 88.9 69.85 180)
+      (effects (font (size 1.27 1.27)) (justify left))
+    )
+    (pin "SATA_B+" input (at 88.9 72.39 180)
+      (effects (font (size 1.27 1.27)) (justify left))
+    )
+    (pin "SATA_B-" input (at 88.9 74.93 180)
+      (effects (font (size 1.27 1.27)) (justify left))
+    )
+    (instances
+      (project "f3_backplane"
+        (path "/a299def6-d097-4d1a-85e0-73dfb51409a1" (page "4"))
+      )
+    )

Commit message: Finish v1.0
Other:
- note added: "F3 Backplane"
- note added: "Mounting Holes"
- title: (none) -> F3 Backplane
- moved on the sheet: H1, H2, H3, H4

Commit message: Add datasheet links and digikey part numbers
Parts:
- H1, H2, H3, H4: now left out of the parts list
Other:
- sheet NVMe SSD ports: added none; removed CLKREQ#, PEWAKE#
Changed lines of the file:
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@@
   )
   (symbol (lib_id "Mechanical:MountingHole_Pad") (at 26.67 165.1 90) (unit 1)
-    (in_bom yes) (on_board yes) (dnp no)
+    (in_bom no) (on_board yes) (dnp no)
     (property "Reference" "H2" (at 26.67 161.29 90)
       (effects (font (size 1.27 1.27)) (justify left))
@@
   )
   (symbol (lib_id "Mechanical:MountingHole_Pad") (at 26.67 152.4 90) (unit 1)
-    (in_bom yes) (on_board yes) (dnp no)
+    (in_bom no) (on_board yes) (dnp no)
     (property "Reference" "H3" (at 26.67 148.59 90)
       (effects (font (size 1.27 1.27)) (justify left))
@@
   )
   (symbol (lib_id "Mechanical:MountingHole_Pad") (at 26.67 177.8 90) (unit 1)
-    (in_bom yes) (on_board yes) (dnp no)
+    (in_bom no) (on_board yes) (dnp no)
     (property "Reference" "H1" (at 26.67 173.99 90)
       (effects (font (size 1.27 1.27)) (justify left))
@@
   )
   (symbol (lib_id "Mechanical:MountingHole_Pad") (at 26.67 139.7 90) (unit 1)
-    (in_bom yes) (on_board yes) (dnp no)
+    (in_bom no) (on_board yes) (dnp no)
     (property "Reference" "H4" (at 26.67 135.89 90)
       (effects (font (size 1.27 1.27)) (justify left))
@@
     )
   )
-  (sheet (at 177.8 100.33) (size 25.4 25.4) (fields_autoplaced)
+  (sheet (at 177.8 100.33) (size 25.4 20.32) (fields_autoplaced)
     (stroke (width 0.1524) (type solid))
     (fill (color 0 0 0 0.0000))
@@
       (effects (font (size 1.27 1.27)) (justify left bottom))
     )
-    (property "Sheetfile" "nvme.kicad_sch" (at 177.8 126.3146 0)
+    (property "Sheetfile" "nvme.kicad_sch" (at 177.8 121.2346 0)
       (effects (font (size 1.27 1.27)) (justify left top))
     )
@@
       (effects (font (size 1.27 1.27)) (justify left))
     )
-    (pin "CLKREQ#" input (at 177.8 123.19 180)
-      (effects (font (size 1.27 1.27)) (justify left))
-    )
-    (pin "PEWAKE#" input (at 177.8 120.65 180)
-      (effects (font (size 1.27 1.27)) (justify left))
-    )
