File: nvme.kicad_sch (KiCad schematic)
At the start: 6 parts, among them J2 Bus_M.2_Socket_M

Commit message: Finish v1.0
Other:
- note added: "M.2 SSD M-Key connector"
- title: (none) -> F3 Backplane NVMe SSD
- moved on the sheet: C1, C2, C3, C4, C5, J2

Commit message: Add datasheet links and digikey part numbers
Parts:
- J2: Digikey Part No. (none) -> MDT420M01001CT-ND
Connections:
- net CLKREQ#: no longer names the net of J2.52 (~{CLKREQ})
- net PEWAKE#: no longer names the net of J2.54 (~{PEWAKE})
- no-connect marks 0 -> 18
Changed lines of the file:
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@@
   (junction (at 107.95 57.15) (diameter 0) (color 0 0 0 0)
   )
+  (no_connect (at 133.35 66.04))
+  (no_connect (at 133.35 83.82))
+  (no_connect (at 133.35 86.36))
+  (no_connect (at 133.35 68.58))
+  (no_connect (at 133.35 96.52))
+  (no_connect (at 133.35 91.44))
+  (no_connect (at 133.35 106.68))
+  (no_connect (at 184.15 134.62))
+  (no_connect (at 133.35 93.98))
+  (no_connect (at 133.35 104.14))
+  (no_connect (at 133.35 88.9))
+  (no_connect (at 133.35 111.76))
+  (no_connect (at 133.35 129.54))
+  (no_connect (at 133.35 101.6))
+  (no_connect (at 184.15 116.84))
+  (no_connect (at 133.35 99.06))
+  (no_connect (at 133.35 109.22))
+  (no_connect (at 184.15 127))
   (wire (pts (xy 125.73 63.5) (xy 133.35 63.5))
     (stroke (width 0) (type default))
@@
     (stroke (width 0) (type default))
   )
-  (wire (pts (xy 125.73 68.58) (xy 133.35 68.58))
-    (stroke (width 0) (type default))
-  )
   (wire (pts (xy 128.27 57.15) (xy 118.11 57.15))
     (stroke (width 0) (type default))
@@
   )
   (wire (pts (xy 148.59 54.61) (xy 148.59 57.15))
-    (stroke (width 0) (type default))
-  )
-  (wire (pts (xy 125.73 66.04) (xy 133.35 66.04))
     (stroke (width 0) (type default))
   )
@@
     (effects (font (size 1.27 1.27)) (justify right))
   )
-  (hierarchical_label "CLKREQ#" (shape input) (at 125.73 66.04 180) (fields_autoplaced)
-    (effects (font (size 1.27 1.27)) (justify right))
-  )
   (hierarchical_label "PERn0" (shape input) (at 125.73 81.28 180) (fields_autoplaced)
     (effects (font (size 1.27 1.27)) (justify right))
@@
   )
   (hierarchical_label "REFCLKn" (shape input) (at 125.73 144.78 180) (fields_autoplaced)
-    (effects (font (size 1.27 1.27)) (justify right))
-  )
-  (hierarchical_label "PEWAKE#" (shape input) (at 125.73 68.58 180) (fields_autoplaced)
     (effects (font (size 1.27 1.27)) (justify right))
   )
@@
       (effects (font (size 1.27 1.27)) hide)
     )
-    (property "Datasheet" "http://read.pudn.com/downloads794/doc/project/3133918/PCIe_M.2_Electromechanical_Spec_Rev1.0_Final_11012013_RS_Clean.pdf#page=155" (at 158.75 80.01 0)
-      (effects (font (size 1.27 1.27)) hide)
-    )
+    (property "Datasheet" "https://cdn.amphenol-cs.com/media/wysiwyg/files/drawing/mdtxxxxxx001.pdf" (at 158.75 80.01 0)
+      (effects (font (size 1.27 1.27)) hide)
+    )
+    (property "Digikey Part No." "MDT420M01001CT-ND" (at 158.75 106.68 0)
+      (effects (font (size 1.27 1.27)) hide)
+    )

Commit message: Fix capacitor values
Parts:
- C1, C2: value 47u -> 47uF
- C3: value 22u -> 22uF
- C4, C5: value 100n -> 100nF
Changed lines of the file:
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@@
       (effects (font (size 1.27 1.27)) (justify left))
     )
-    (property "Value" "47u" (at 120.65 53.34 0)
+    (property "Value" "47uF" (at 120.65 53.34 0)
       (effects (font (size 1.27 1.27)) (justify left))
     )
@@
       (effects (font (size 1.27 1.27)) (justify left))
     )
-    (property "Value" "100n" (at 151.13 53.34 0)
+    (property "Value" "100nF" (at 151.13 53.34 0)
       (effects (font (size 1.27 1.27)) (justify left))
     )
@@
       (effects (font (size 1.27 1.27)) (justify left))
     )
-    (property "Value" "22u" (at 130.81 53.34 0)
+    (property "Value" "22uF" (at 130.81 53.34 0)
       (effects (font (size 1.27 1.27)) (justify left))
     )
@@
       (effects (font (size 1.27 1.27)) (justify left))
     )
-    (property "Value" "100n" (at 140.97 53.34 0)
+    (property "Value" "100nF" (at 140.97 53.34 0)
       (effects (font (size 1.27 1.27)) (justify left))
     )
@@
       (effects (font (size 1.27 1.27)) (justify left))
     )
-    (property "Value" "47u" (at 110.49 53.34 0)
-      (effects (font (size 1.27 1.27)) (justify left))
-    )
+    (property "Value" "47uF" (at 110.49 53.34 0)
+      (effects (font (size 1.27 1.27)) (justify left))
+    )
